Commit message: Changed URDF Files

File: Robor/urdf/Robor.urdf (robot description, URDF)
Before this commit: robot Robor, 4 links, 3 joints
Links:
- link Castor Wheel: mass 0.5 -> 0.30661
Joints:
- joint CW: axis 0 1 0 -> 0 0 0; limit lower=0 upper=0 effort=0 velocity=0 -> (none); origin xyz=-0.15394 -0.35895 0.2043 rpy=-1.5735 0.069867 -0.03916 -> xyz=-0.16947 -0.36094 0.20391 rpy=1.5708 0.10274 0; type continuous -> fixed
