Commit message: updated model urdf with gazebo plugin.

File: urdf/Robor.urdf (robot description, URDF)
Before this commit: robot Robor, 4 links, 3 joints
Links:
- added link Castor Frame, mass 0.12593; collision mesh filename=package://Robor/meshes/Castor Frame.STL; visual mesh filename=package://Robor/meshes/Castor Frame.STL
- link Castor Wheel: mass 0.30661 -> 0.18068
Joints:
- removed joint CW
- added joint CWF: type revolute, parent Chassis, child Castor Frame, origin xyz=-0.13379 -0.42645 0.17915 rpy=1.5708 0 0, axis 0 0 1, limit lower=0 upper=0 effort=0 velocity=0
- added joint CWW: type continuous, parent Castor Frame, child Castor Wheel, origin xyz=-0.035684 0.024756 -0.065505 rpy=0 0 -0.10274, axis 0.10256 -0.99473 0
- joint LW: origin xyz=0.11841 -0.39765 0.35775 rpy=1.5708 0 2.7649 -> xyz=0.11841 -0.39765 0.35775 rpy=1.5708 0 -0.37673
- joint RW: axis 0 1 0 -> 0 -1 0
