Commit message: lidar plugin working.

File: urdf/modbot_without.urdf (robot description, URDF)
Before this commit: robot modbot, 5 links, 4 joints
Links:
- added link Lidar, mass 10.42; collision mesh filename=package://modbot/meshes/meshes_without/Lidar.STL; visual mesh filename=package://modbot/meshes/meshes_without/Lidar.STL
- link Caster Frame: geometry collision mesh filename=package://modbot/meshes/meshes_without/Caster Frame.STL; visual mesh filename=package://modbot/meshes/meshes_without/Caster Frame.STL
- link Caster Wheel: geometry collision mesh filename=package://modbot/meshes/meshes_without/Caster Wheel.STL; visual mesh filename=package://modbot/meshes/meshes_without/Caster Wheel.STL
- link Chassis: mass 10.493 -> 10.42; geometry collision mesh filename=package://modbot/meshes/meshes_without/Chassis.STL; visual mesh filename=package://modbot/meshes/meshes_without/Chassis.STL
- link Left Wheel: geometry collision mesh filename=package://modbot/meshes/meshes_without/Left Wheel.STL; visual mesh filename=package://modbot/meshes/meshes_without/Left Wheel.STL
- link Right Wheel: geometry collision mesh filename=package://modbot/meshes/meshes_without/Right Wheel.STL; visual mesh filename=package://modbot/meshes/meshes_without/Right Wheel.STL
Joints:
- added joint L: type fixed, parent Chassis, child Lidar, origin xyz=-0.048789 -0.080754 0.31207 rpy=3.1416 0 0, axis 0 0 0
- joint CWW: origin xyz=-0.0125 0 -0.0675 rpy=0 0 0 -> xyz=-0.0125000000000001 0 -0.0674999999999999 rpy=0 0 0
