Commit message: fixed lidar sensor and its working fine now.

File: urdf/modbot.urdf (robot description, URDF)
Before this commit: robot modbot, 5 links, 4 joints
Links:
- added link Lidar, mass 0.073085; collision mesh filename=package://modbot/meshes/Lidar.STL; visual mesh filename=package://modbot/meshes/Lidar.STL
- link Caster Frame: geometry collision mesh filename=package://modbot/meshes/Caster Frame.STL; visual mesh filename=package://modbot/meshes/Caster Frame.STL
- link Caster Wheel: geometry collision mesh filename=package://modbot/meshes/Caster Wheel.STL; visual mesh filename=package://modbot/meshes/Caster Wheel.STL
- link Chassis: mass 10.493 -> 10.42; geometry collision mesh filename=package://modbot/meshes/Chassis.STL; visual mesh filename=package://modbot/meshes/Chassis.STL
- link Left Wheel: geometry collision mesh filename=package://modbot/meshes/Left Wheel.STL; visual mesh filename=package://modbot/meshes/Left Wheel.STL
- link Right Wheel: geometry collision mesh filename=package://modbot/meshes/Right Wheel.STL; visual mesh filename=package://modbot/meshes/Right Wheel.STL
Joints:
- added joint L: type fixed, parent Chassis, child Lidar, origin xyz=0.18573 -0.8271 0.17915 rpy=1.5708 0 0, axis 0 0 0

Commit message: fixed drifting of the robot by new inertial values.

File: urdf/modbot.urdf (robot description, URDF)
Before this commit: robot modbot, 6 links, 5 joints
Links:
- link Caster Frame: mass 0.069072 -> 0.5
- link Caster Wheel: mass 0.19827 -> 0.5
- link Chassis: mass 10.42 -> 17.5
- link Left Wheel: mass 0.72827 -> 2
- link Lidar: mass 0.073085 -> 0.1
- link Right Wheel: mass 0.72827 -> 2
Joints:
- joint CWF: origin xyz=-0.13379 -0.42645 0.17915 rpy=1.5708 0 0 -> xyz=-0.1636 0 -0.0492 rpy=0 0 0
- joint L: origin xyz=0.18573 -0.8271 0.17915 rpy=1.5708 0 0 -> xyz=0.15592 0 0.35145 rpy=0 0 0
- joint LW: origin xyz=0.11841 -0.39765 0.35775 rpy=1.5708 0 -0.37673 -> xyz=0.0886 0.1786 -0.078 rpy=0 -0.37673 0
- joint RW: origin xyz=0.11841 -0.39765 0 rpy=-1.5708 0 0.78245 -> xyz=0.0886 -0.17915 -0.078 rpy=3.1416 0.78245 0

Commit message: visualising modbot in rviz.

File: urdf/modbot.urdf (robot description, URDF)
Before this commit: robot modbot, 6 links, 5 joints
Links:
- link Caster Frame: mass 0.5 -> 0.069072
- link Caster Wheel: mass 0.5 -> 0.19827
- link Chassis: mass 17.5 -> 10.42
- link Lidar: mass 0.1 -> 0
Joints:
- joint RW: origin xyz=0.0886 -0.17915 -0.078 rpy=3.1416 0.78245 0 -> xyz=0.0886 -0.17915 -0.078 rpy=0 -0.78245 3.1416
